Commit message: Refactor ros2_control configuration to support dynamic prefix
Signed-off-by: Baoan Du <baoan.du.xj@renesas.com>

File: urdf/inspire_rh56_hand_left.urdf.xacro (robot description, xacro)
@@ -9,8 +9,9 @@
   <xacro:arg name="baudrate" default="115200"/>
   <xacro:arg name="use_mock_hardware" default="false"/>
+  <xacro:arg name="prefix" default=""/>
   <!-- World link -->
   <link name="world"/>
   <!-- Instantiate the left hand -->
-  <xacro:inspire_hand_left parent="world" prefix="">
+  <xacro:inspire_hand_left parent="world" prefix="$(arg prefix)">
     <origin xyz="0 0 0" rpy="0 0 0"/>
   </xacro:inspire_hand_left>
@@ -21,3 +22,4 @@
     baudrate="$(arg baudrate)"
     use_mock_hardware="$(arg use_mock_hardware)"
+    prefix="$(arg prefix)"
   /></robot>

File: urdf/inspire_rh56_hand_macro.ros2_control.xacro (robot description, xacro)
@@ -1,16 +1,22 @@
 <?xml version="1.0"?>
 <robot xmlns:xacro="http://www.ros.org/wiki/xacro">
+  <!--
+    ROS 2 Control macro for Inspire RH56 Hand
+    This macro adds ros2_control tags to the robot description
+    Supports both real hardware and mock hardware configurations
+  -->
   <xacro:macro name="inspire_rh56_hand_ros2_control" params="
-    name
+    name:=inspire_rh56_hand
     serial_port:=/dev/ttyUSB0
     baudrate:=115200
     use_mock_hardware:=false
+    prefix:=''
     ">
-    <ros2_control name="${name}" type="system" rw_rate="50">
-      <!-- Hardware interface plugin -->
+    <ros2_control name="${prefix}${name}" type="system" rw_rate="50">
+      <!-- Hardware interface plugin chosen conditionally -->
       <hardware>
         <xacro:if value="${use_mock_hardware}">
           <plugin>mock_components/GenericSystem</plugin>
-          <param name="state_following_offset">0.0</param>
+          <param name="position_state_following_offset">0.0</param>
         </xacro:if>
         <xacro:unless value="${use_mock_hardware}">
@@ -22,5 +28,5 @@
       <!-- Joint definitions -->
       <!-- Thumb joints -->
-      <joint name="thumb_proximal_yaw_joint">
+      <joint name="${prefix}thumb_proximal_yaw_joint">
         <command_interface name="position">
           <param name="min">0.0</param>
@@ -30,5 +36,5 @@
         <state_interface name="velocity"/>
       </joint>
-      <joint name="thumb_proximal_pitch_joint">
+      <joint name="${prefix}thumb_proximal_pitch_joint">
         <command_interface name="position">
           <param name="min">0.0</param>
@@ -39,5 +45,5 @@
       </joint>
       <!-- Four finger joints -->
-      <joint name="index_proximal_joint">
+      <joint name="${prefix}index_proximal_joint">
         <command_interface name="position">
           <param name="min">0.0</param>
@@ -47,5 +53,5 @@
         <state_interface name="velocity"/>
       </joint>
-      <joint name="middle_proximal_joint">
+      <joint name="${prefix}middle_proximal_joint">
         <command_interface name="position">
           <param name="min">0.0</param>
@@ -55,5 +61,5 @@
         <state_interface name="velocity"/>
       </joint>
-      <joint name="ring_proximal_joint">
+      <joint name="${prefix}ring_proximal_joint">
         <command_interface name="position">
           <param name="min">0.0</param>
@@ -63,5 +69,5 @@
         <state_interface name="velocity"/>
       </joint>
-      <joint name="pinky_proximal_joint">
+      <joint name="${prefix}pinky_proximal_joint">
         <command_interface name="position">
           <param name="min">0.0</param>

File: urdf/inspire_rh56_hand_right.urdf.xacro (robot description, xacro)
@@ -9,8 +9,9 @@
   <xacro:arg name="baudrate" default="115200"/>
   <xacro:arg name="use_mock_hardware" default="false"/>
+  <xacro:arg name="prefix" default=""/>
   <!-- World link -->
   <link name="world"/>
   <!-- Instantiate the right hand -->
-  <xacro:inspire_hand_right parent="world" prefix="">
+  <xacro:inspire_hand_right parent="world" prefix="$(arg prefix)">
     <origin xyz="0 0 0" rpy="0 0 0"/>
   </xacro:inspire_hand_right>
@@ -21,3 +22,4 @@
     baudrate="$(arg baudrate)"
     use_mock_hardware="$(arg use_mock_hardware)"
+    prefix="$(arg prefix)"
   /></robot>
